File: hardware/kicad/TinyDyno.kicad_pcb (KiCad board)
At the start: 2 copper layers, 72 x 72 mm, 35 parts, among them J1 TYPE-C-31-M-12, SW1 TS-1187A-B-A-B, SW2 TS-1187A-B-A-B, U1 LR1107G-33, U2 LR1107G-33, U3 INA228, U4 ESP32-S3-WROOM-1-N16R8, U5 LSM6DS3TR-C

Commit message: finished pcb
Parts:
- U3: value INA228 -> INA226
- moved C2 6.00 mm to (105.2, 121.6), turned to 0 degrees
- turned U5 to 90 degrees
Connections:
- R8 pad 1: /3V3_MEAS -> /3V3_PERIPH
Routing:
- net /3V3_PERIPH: track 0.00 -> 139.2 mm, vias 0 -> 4
- net +5V: track 0.00 -> 74.2 mm, vias 0 -> 2
- net /USB_DN: track 0.00 -> 49.1 mm, vias 0 -> 2
- net /USB_DP: track 0.00 -> 44.6 mm
- net Net-(U4-EN): track 0.00 -> 44.4 mm
- net GND: track 0.00 -> 34.0 mm, vias 0 -> 30
- net /3V3_MEAS: track 0.00 -> 26.3 mm, vias 0 -> 2
- net /INA_ALERT: track 0.00 -> 23.6 mm, vias 0 -> 2
- net /I2C_SDA: track 0.00 -> 21.1 mm, vias 0 -> 3
- net /I2C_SCL: track 0.00 -> 19.3 mm, vias 0 -> 4
- net /SENSE_P: track 0.00 -> 16.3 mm, vias 0 -> 2
- net /3V3_REGA: track 0.00 -> 14.1 mm
- net Net-(U4-IO0): track 0.00 -> 13.1 mm
- net /IMU_INT1: track 0.00 -> 12.3 mm
- net /MIC_DATA: track 0.00 -> 11.5 mm, vias 0 -> 2
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- added copper zone on B.Cu, net GND
- added copper zone on F.Cu, net GND
