File: hardware/kicad/TinyDyno.kicad_sch (KiCad schematic)
At the start: 0 parts

Commit message: half baked schematic
Parts:
- added C1: 1u, Capacitor_SMD:C_0603_1608Metric, symbol Device:C
- added C2: 22u, Capacitor_SMD:C_0603_1608Metric, symbol Device:C
- added C3: 1u, Capacitor_SMD:C_0805_2012Metric, symbol Device:C
- added C4: 22u, Capacitor_SMD:C_0805_2012Metric, symbol Device:C
- added C5: 100n, Capacitor_SMD:C_0603_1608Metric, symbol Device:C
- added J1: TYPE-C-31-M-12, Connector_USB:USB_C_Receptacle_HRO_TYPE-C-31-M-12, symbol Connector:USB_C_Receptacle_USB2.0_16P
- added JP1: SJ, Jumper:SolderJumper-2_P1.3mm_Bridged_RoundedPad1.0x1.5mm, symbol Jumper:SolderJumper_2_Bridged
- added R1, R2: 5.1k, Resistor_SMD:R_0603_1608Metric, symbol Device:R
- added R3: 75m, Resistor_SMD:R_2512_6332Metric, symbol Device:R
- added R4, R5, R6: 4.7k, Resistor_SMD:R_0603_1608Metric, symbol Device:R
- added U1, U2: LR1107G-33, Package_TO_SOT_SMD:SOT-223-3_TabPin2, symbol Regulator_Linear:AMS1117-3.3
- added U3: INA228, Package_SO:TSSOP-10_3x3mm_P0.5mm, symbol Sensor_Energy:INA228
Connections:
- new net: J1.A5 (CC1), R1.1
- new net: J1.B5 (CC2), R2.1
- new net +5V: C1.1, C3.1, J1.A4 (VBUS), J1.A9 (VBUS), J1.B4 (VBUS), J1.B9 (VBUS), U1.3 (VI), U2.3 (VI)
- new net 3V3_MAES: R3.2, U3.8 (Vbus), U3.9 (Vin-)
- new net 3V3_PERIPH: C2.1, C5.1, R4.1, R5.1, R6.1, U1.2 (VO), U3.6 (VS)
- new net 3V3_REGA: C4.1, JP1.1 (A), U2.2 (VO)
- new net GND: C1.2, C2.2, C3.2, C4.2, C5.2, J1.A1 (GND), J1.A12 (GND), J1.B1 (GND), J1.B12 (GND), J1.SH (SHIELD), R1.2, R2.2, U1.1 (GND), U2.1 (GND), U3.1 (A1), U3.2 (A0), U3.7 (GND)
- new net I2C_SCL: R4.2, U3.5 (SCL)
- new net I2C_SDA: R5.2, U3.4 (SDA)
- new net INA_ALERT: R6.2, U3.3 (~{Alert})
- new net SENSE_P: JP1.2 (B), R3.1, U3.10 (Vin+)
- new net USB_DN: J1.A7 (D-), J1.B7 (D-)
- new net USB_DP: J1.A6 (D+), J1.B6 (D+)
- no-connect marks 0 -> 2
Other:
- title: (none) -> TinyDyno

Commit message: Schematic done
Finished the schematic
Parts:
- added C10, C11, C7, C9: 100n, Capacitor_SMD:C_0603_1608Metric, symbol Device:C
- added C6: 22u, Capacitor_SMD:C_0805_2012Metric, symbol Device:C
- added C8: 1u, Capacitor_SMD:C_0603_1608Metric, symbol Device:C
- added D1: KT-0603R, LED_SMD:LED_0603_1608Metric, symbol Device:LED
- added MK1: IM69D130V01, Sensor_Audio:Infineon_PG-LLGA-5-1, symbol Sensor_Audio:IM69D130
- added R10: 1k, Resistor_SMD:R_0603_1608Metric, symbol Device:R
- added R11, R9: 22, Resistor_SMD:R_0603_1608Metric, symbol Device:R
- added R7, R8: 10k, Resistor_SMD:R_0603_1608Metric, symbol Device:R
- added SW1: TS-1187A-B-A-B, Button_Switch_THT:SW_NKK_GW12LJP, symbol Switch:SW_Push
- added SW2: TS-1187A-B-A-B, Button_Switch_SMD:SW_Push_1P1T_XKB_TS-1187A, symbol Switch:SW_Push
- added TP1, TP2: TestPoint, TestPoint:TestPoint_Pad_D1.5mm, symbol Connector:TestPoint
- added U4: ESP32-S3-WROOM-1-N16R8, RF_Module:ESP32-S3-WROOM-1, symbol RF_Module:ESP32-S3-WROOM-1
- added U5: LSM6DS3TR-C, Package_LGA:LGA-14_3x2.5mm_P0.5mm_LayoutBorder3x4y, symbol Sensor_Motion:LSM6DS3
- R4, R5, R6: value 4.7k -> 5.1k
Connections:
- net 3V3_PERIPH: now also C10.1, C11.1, C9.1, D1.2 (A), MK1.2 (VDD), U5.12 (CS), U5.5 (VDDIO), U5.8 (VDD)
- net GND: now also C10.2, C11.2, C6.2, C7.2, C8.2, C9.2, MK1.4 (SELECT), MK1.5 (GND), SW1.1, SW2.1, TP2.1, U4.1 (GND), U4.40 (GND), U4.41 (GND), U5.1 (SDO/SA0), U5.2 (SDX), U5.3 (SCX), U5.6 (GND), U5.7 (GND)
- net I2C_SCL: now also U4.5 (IO5), U5.13 (SCL)
- net I2C_SDA: now also U4.4 (IO4), U5.14 (SDA)
- net INA_ALERT: now also U4.6 (IO6)
- net USB_DN: now also R11.2
- net USB_DP: now also R9.2
- net 3V3_MAES renamed 3V3_MEAS
- net 3V3_MEAS: now also C6.1, C7.1, R7.1, R8.1, U4.2 (3V3)
- new net: D1.1 (K), R10.1
- new net: R10.2, U4.38 (IO2)
- new net: C8.1, R7.2, SW1.2, U4.3 (EN)
- new net: R11.1, U4.13 (USB_D-)
- new net: R9.1, U4.14 (USB_D+)
- new net: R8.2, SW2.2, U4.27 (IO0)
- new net IMU_INT1: U4.7 (IO7), U5.4 (INT1)
- new net MIC_CLK: MK1.3 (CLOCK), U4.35 (IO42)
- new net MIC_DATA: MK1.1 (DATA), U4.34 (IO41)
- new net TEST_MARK: TP1.1, U4.39 (IO1)
- no-connect marks 2 -> 28
Other:
- moved on the sheet: C1, C2, C3, C4, C5, J1, JP1, R1, R2, R3, R4, R5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

Commit message: fixed footprints
fixed the footprints of capacitors
Parts:
- C2: footprint Capacitor_SMD:C_0603_1608Metric -> Capacitor_SMD:C_0805_2012Metric
- C3: footprint Capacitor_SMD:C_0805_2012Metric -> Capacitor_SMD:C_0603_1608Metric
Changed lines of the file:
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@@
 			)
 		)
-		(property "Footprint" "Capacitor_SMD:C_0603_1608Metric"
+		(property "Footprint" "Capacitor_SMD:C_0805_2012Metric"
 			(at 246.0752 140.97 0)
 			(hide yes)
@@
 			)
 		)
-		(property "Footprint" "Capacitor_SMD:C_0805_2012Metric"
+		(property "Footprint" "Capacitor_SMD:C_0603_1608Metric"
 			(at 230.8352 167.64 0)
 			(hide yes)

Commit message: fixed bom
deleted test points from bom
Parts:
- SW1: footprint Button_Switch_THT:SW_NKK_GW12LJP -> Button_Switch_SMD:SW_Push_1P1T_XKB_TS-1187A
- TP1, TP2: now left out of the parts list
Changed lines of the file:
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@@
 		(body_style 1)
 		(exclude_from_sim no)
-		(in_bom yes)
+		(in_bom no)
 		(on_board yes)
 		(in_pos_files yes)
@@
 		(body_style 1)
 		(exclude_from_sim no)
-		(in_bom yes)
+		(in_bom no)
 		(on_board yes)
 		(in_pos_files yes)
@@
 			)
 		)
-		(property "Footprint" "Button_Switch_THT:SW_NKK_GW12LJP"
+		(property "Footprint" "Button_Switch_SMD:SW_Push_1P1T_XKB_TS-1187A"
 			(at 80.01 114.3 0)
 			(hide yes)

Commit message: placement
Parts:
- C1, C3, C8: LCSC (none) -> C15849
- C10, C11, C5, C7, C9: LCSC (none) -> C14663
- C2, C4, C6: LCSC (none) -> C45783
- D1: LCSC (none) -> C2286
- J1: LCSC (none) -> C165948
- MK1: LCSC (none) -> C536262
- R1, R2, R4, R5, R6: LCSC (none) -> C23186
- R10: LCSC (none) -> C21190
- R11, R9: LCSC (none) -> C23345
- R3: LCSC (none) -> C76252
- R7, R8: LCSC (none) -> C25804
- SW1, SW2: LCSC (none) -> C318884
- U1, U2: LCSC (none) -> C171499
- U3: LCSC (none) -> C2887910
- U4: LCSC (none) -> C2913202
- U5: LCSC (none) -> C967633

Commit message: finished pcb
Parts:
- U3: value INA228 -> INA226; LCSC C2887910 -> C49851
Connections:
- net 3V3_MEAS: no longer R8.1
- net 3V3_PERIPH: now also R8.1
Changed lines of the file:
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@@
 		)
 	)
-	(label "3V3_MEAS"
+	(label "3V3_PERIPH"
 		(at 68.58 111.76 90)
 		(effects
@@
 			)
 		)
-		(property "Value" "INA228"
+		(property "Value" "INA226"
 			(at 280.2733 135.89 0)
 			(show_name no)
@@
 			)
 		)
-		(property "LCSC" " C2887910"
+		(property "LCSC" " C49851"
 			(at 278.13 148.59 0)
 			(hide yes)
